File: remote control/Conectores.sch (EAGLE design)
At the start: 31 parts, among them X2 SSW-110-02-S-S, X5 SSW-110-02-S-S, X6 SSW-120-02-S-S, X7 SSW-120-02-S-S

Commit message: Remote Control almost final version
Parts:
- removed IC1: (no value), ic-package:DIL40
- removed X2, X5: SSW-110-02-S-S, con-samtec:SSW-110-02-S-S
- removed X6, X7: SSW-120-02-S-S, con-samtec:SSW-120-02-S-S
- added C6: 100n, rcl:C-EUC0805
- added C7: 1u, rcl:CPOL-EUCT3528
- added CONECTOR_FRONT1, CONNECTOR_REAR1: (no value), con-ml:ML40
- added FL_CHIP, FR_CHIP, MAIN_CHIP, RL_CHIP, RR_CHIP: (no value), ic-package:DIL40
- added JP1, JP2: (no value), pinhead-2:PINHD-1X10_2.00
- added LED10, LED11, LED12, LED13, LED14, LED6, LED7, LED8, LED9: LG_T679-E1F1-1, led:LG_T679-E1F1-1
- added Q10, Q11, Q3, Q4, Q5, Q6, Q7, Q8, Q9: (no value), semicon-smd-ipc:NPN-TRANSISTOR_SOT23
- added R13: 60, rcl:R-EU_R0805
- added R14, R15, R16, R17, R18, R19, R20, R21, R22, R23, R24: (no value), rcl:R-EU_R0805
- added R25, R26, R27, R28, R29, R30, R31, R32, R33, R34, R35: 330, rcl:R-EU_R0805
- added S1: (no value), switch-omron:10-XX
- C2: value 10u -> 4u7; device rcl:CPOL-EUCT3528 -> rcl:CPOL-EUSMCE
- C3: value 4u7 -> 100n; device rcl:CPOL-EUSMCE -> rcl:C-EUC0805K
- LED1, LED3, LED4, LED5: value (none) -> LG_T679-E1F1-1; device led:LEDP-LCC-2 -> led:LG_T679-E1F1-1
- R1: value 330 -> 100; device rcl:R-EU_M0805 -> resistor:R-EU_M0805
- R10: value 1K8 -> 10k
- R11: value 10k -> 220; device rcl:R-EU_M0805 -> rcl:R-EU_R0805
- R12: value 10K -> 330; device rcl:R-EU_M0805 -> rcl:R-EU_R0805
- R2: value 220 -> 10K; device rcl:R-EU_M0805 -> resistor:R-EU_M0805
- R3: value 330 -> 3K3; device rcl:R-EU_M0805 -> resistor:R-EU_M0805
- R4: value 330 -> 1K8; device rcl:R-EU_M0805 -> resistor:R-EU_M0805
- R5: value 10k -> 470; device rcl:R-EU_M0805 -> resistor:R-EU_M0805
- R6: value 100 -> 10k
- R7: value 10K -> 10k
- R8: value 470 -> 10k
- R9: value 3K3 -> 10k
- X3: device con-ptr500:AK300/4 -> con-ptr500:AK300/2
- X4: device con-ptr500:AK300/2 -> con-subd:F09HP
Connections:
- removed net 3V3: DC2.VOUT, R2.2, R7.1, X2-1.1
- removed net 5V: C2.+, DC1.VOUT, IC1.40, R1.2, R12.1, R3.2, R4.2, X3-1.KL, X6-2.1
- removed net I2C_CLOCK: IC1.7, X3-2.KL
- removed net I2C_DATA: IC1.8, X3-3.KL
- removed net LED1: IC1.9, R5.2
- removed net LED2: IC1.10, R11.2
- removed net MISO: IC1.38, X6-8.1
- removed net MOSI: IC1.37, X6-7.1
- removed net SCK: IC1.39, X6-9.1
- removed net SS: IC1.36, X6-6.1
- removed net XBEELED1: LED2.C, X2-6.1
- removed net XBEERESET1: R7.2, X2-5.1
- new net CAN_H: FL_CHIP.19, FR_CHIP.19, MAIN_CHIP.19, R13.2, RL_CHIP.19, RR_CHIP.19, X4.7
- new net CAN_L: FL_CHIP.18, FR_CHIP.18, MAIN_CHIP.18, R13.1, RL_CHIP.18, RR_CHIP.18, X4.2
- new net FL_AI0: CONECTOR_FRONT1.33, FL_CHIP.26
- new net FL_AI1: CONECTOR_FRONT1.34, FL_CHIP.25
- new net FL_AI2: CONECTOR_FRONT1.35, FL_CHIP.24
- new net FL_AI3: CONECTOR_FRONT1.40, FL_CHIP.23
- new net FL_DI0: CONECTOR_FRONT1.11, FL_CHIP.13
- new net FL_DI1: CONECTOR_FRONT1.13, FL_CHIP.14
- new net FL_DO0: CONECTOR_FRONT1.6, FL_CHIP.38
- new net FL_DO1: CONECTOR_FRONT1.7, FL_CHIP.37
- new net FL_DO2: CONECTOR_FRONT1.8, FL_CHIP.36
- new net FL_LED1: FL_CHIP.33, R24.1
- new net FL_LED2: FL_CHIP.32, R23.1
- new net FL_PWM0: CONECTOR_FRONT1.21, FL_CHIP.7
- new net FL_PWM1: CONECTOR_FRONT1.22, FL_CHIP.8
- new net FL_PWM2: CONECTOR_FRONT1.23, FL_CHIP.9
- new net FL_PWM3: CONECTOR_FRONT1.24, FL_CHIP.10
- new net FL_PWM4: CONECTOR_FRONT1.25, FL_CHIP.11
- new net FL_PWM5: CONECTOR_FRONT1.26, FL_CHIP.12
- new net FR_AI0: CONECTOR_FRONT1.37, FR_CHIP.26
- new net FR_AI1: CONECTOR_FRONT1.38, FR_CHIP.25
- new net FR_AI2: CONECTOR_FRONT1.39, FR_CHIP.24
- new net FR_AI3: CONECTOR_FRONT1.36, FR_CHIP.23
- new net FR_DI0: CONECTOR_FRONT1.12, FR_CHIP.13
- new net FR_DI1: CONECTOR_FRONT1.14, FR_CHIP.14
- new net FR_DIP2: FR_CHIP.29, R7.1
- new net FR_DO0: CONECTOR_FRONT1.3, FR_CHIP.38
- new net FR_DO1: CONECTOR_FRONT1.4, FR_CHIP.37
- new net FR_DO2: CONECTOR_FRONT1.5, FR_CHIP.36
- new net FR_LED1: FR_CHIP.33, R14.1
- new net FR_LED2: FR_CHIP.32, R15.1
- new net FR_PWM0: CONECTOR_FRONT1.15, FR_CHIP.7
- new net FR_PWM1: CONECTOR_FRONT1.16, FR_CHIP.8
- new net FR_PWM2: CONECTOR_FRONT1.17, FR_CHIP.9
- new net FR_PWM3: CONECTOR_FRONT1.18, FR_CHIP.10
- new net FR_PWM4: CONECTOR_FRONT1.19, FR_CHIP.11
- new net FR_PWM5: CONECTOR_FRONT1.20, FR_CHIP.12
- new net LED: JP1.6, LED1.C
- new net MAIN_LED1: MAIN_CHIP.7, R18.1
- new net MAIN_LED2: MAIN_CHIP.8, R19.1
- new net MAIN_LED3: MAIN_CHIP.9, R20.1
- new net N$11: Q1.B, R24.2
- new net N$12: Q2.B, R23.2
- new net N$14: LED5.C, Q5.C
- new net N$15: LED8.C, Q9.C
- new net N$16: LED10.C, Q11.C
- new net N$17: LED11.C, Q7.C
- new net N$18: LED13.C, Q3.C
- new net N$19: LED7.C, Q2.C
- new net N$20: LED14.C, Q4.C
- new net N$21: LED6.C, Q6.C
- new net N$22: LED12.C, Q8.C
- new net N$23: LED9.C, Q10.C
- new net N$24: LED5.A, R25.1
- new net N$25: LED6.A, R26.1
- new net N$26: LED8.A, R27.1
- new net N$27: LED9.A, R28.1
- new net N$28: LED10.A, R29.1
- new net N$29: LED12.A, R30.1
- new net N$30: LED11.A, R31.1
- new net N$31: LED14.A, R32.1
- new net N$32: LED13.A, R33.1
- new net N$33: LED4.A, R34.1
- new net N$34: LED7.A, R35.1
- new net N$35: Q9.B, R18.2
- new net N$36: Q10.B, R19.2
- new net N$38: Q11.B, R20.2
- new net N$5: Q5.B, R14.2
- new net RESET: C3.1, FL_CHIP.3, FR_CHIP.3, MAIN_CHIP.3, RL_CHIP.3, RR_CHIP.3, S1.S, S1.S1
- new net RL_AI0: CONNECTOR_REAR1.37, RL_CHIP.26
- new net RL_AI1: CONNECTOR_REAR1.38, RL_CHIP.25
- new net RL_AI2: CONNECTOR_REAR1.39, RL_CHIP.24
- new net RL_AI3: CONNECTOR_REAR1.36, RL_CHIP.23
- new net RL_DI0: CONNECTOR_REAR1.12, RL_CHIP.13
- new net RL_DI1: CONNECTOR_REAR1.14, RL_CHIP.14
- new net RL_DIP2: R8.1, RL_CHIP.29
- new net RL_DIP3: R9.1, RL_CHIP.28
- new net RL_DO0: CONNECTOR_REAR1.3, RL_CHIP.38
- new net RL_DO1: CONNECTOR_REAR1.4, RL_CHIP.37
- new net RL_DO2: CONNECTOR_REAR1.5, RL_CHIP.36
- new net RL_LED1: R21.1, RL_CHIP.33
- new net RL_LED2: R22.1, RL_CHIP.32
- new net RL_PWM0: CONNECTOR_REAR1.15, RL_CHIP.7
- new net RL_PWM1: CONNECTOR_REAR1.16, RL_CHIP.8
- new net RL_PWM2: CONNECTOR_REAR1.17, RL_CHIP.9
- new net RL_PWM3: CONNECTOR_REAR1.18, RL_CHIP.10
- new net RL_PWM4: CONNECTOR_REAR1.19, RL_CHIP.11
- new net RL_PWM5: CONNECTOR_REAR1.20, RL_CHIP.12
- new net RR_AI0: CONNECTOR_REAR1.33, RR_CHIP.26
- new net RR_AI1: CONNECTOR_REAR1.34, RR_CHIP.25
- new net RR_AI2: CONNECTOR_REAR1.35, RR_CHIP.24
- new net RR_AI3: CONNECTOR_REAR1.40, RR_CHIP.23
- new net RR_DI0: CONNECTOR_REAR1.11, RR_CHIP.13
- new net RR_DI1: CONNECTOR_REAR1.13, RR_CHIP.14
- new net RR_DIP1: R10.1, RR_CHIP.30
- new net RR_DO0: CONNECTOR_REAR1.6, RR_CHIP.38
- new net RR_DO1: CONNECTOR_REAR1.7, RR_CHIP.37
- new net RR_DO2: CONNECTOR_REAR1.8, RR_CHIP.36
- new net RR_LED1: R17.1, RR_CHIP.33
- new net RR_LED2: R16.1, RR_CHIP.32
- new net RR_PWM0: CONNECTOR_REAR1.21, RR_CHIP.7
- new net RR_PWM1: CONNECTOR_REAR1.22, RR_CHIP.8
- new net RR_PWM2: CONNECTOR_REAR1.23, RR_CHIP.9
- new net RR_PWM3: CONNECTOR_REAR1.24, RR_CHIP.10
- new net RR_PWM4: CONNECTOR_REAR1.25, RR_CHIP.11
- new net RR_PWM5: CONNECTOR_REAR1.26, RR_CHIP.12
- new net VCC: DC1.VOUT, FL_CHIP.40, FR_CHIP.40, LED2.A, MAIN_CHIP.40, R10.2, R25.2, R26.2, R27.2, R28.2, R29.2, R30.2, R31.2, R32.2, R33.2, R34.2, R35.2, R6.2, R7.2, R8.2, R9.2, RL_CHIP.40, RR_CHIP.40
- new net VCC3V3: C6.1, C7.+, DC2.VOUT, JP1.1, LED3.A, R2.1
- new net XBEERESET: JP1.5, R2.2
- net GND: now also C3.2, C6.2, C7.-, CONECTOR_FRONT1.10, CONECTOR_FRONT1.27, CONECTOR_FRONT1.28, CONECTOR_FRONT1.31, CONECTOR_FRONT1.32, CONNECTOR_REAR1.10, CONNECTOR_REAR1.27, CONNECTOR_REAR1.28, CONNECTOR_REAR1.31, CONNECTOR_REAR1.32, FL_CHIP.20, FL_CHIP.29, FL_CHIP.30, FR_CHIP.20, FR_CHIP.28, FR_CHIP.30, JP1.10, MAIN_CHIP.20, MAIN_CHIP.28, MAIN_CHIP.29, MAIN_CHIP.30, Q10.E, Q11.E, Q3.E, Q4.E, Q5.E, Q6.E, Q7.E, Q8.E, Q9.E, R11.2, R12.2, R3.2, R5.1, RL_CHIP.20, RL_CHIP.30, RR_CHIP.20, RR_CHIP.28, RR_CHIP.29, S1.P, S1.P1, X3-2.KL; no longer C3.-, IC1.20, LED1.C, LED3.C, R8.1, R9.2, X2-10.1, X3-4.KL, X4-1.KL, X6-1.1, X6-11.1
- net N$1: now also LED1.A, R5.2; no longer LED2.A, R8.2
- net N$10: now also Q4.B, R22.2; no longer R12.2, X6-5.1
- net N$2: now also LED3.C, R11.1; no longer LED1.A, R1.1
- net N$3: now also FL_CHIP.28, R6.1; no longer LED3.A, R2.1
- net N$4: now also LED2.C, R12.1; no longer LED4.A, R3.1
- net N$6: now also Q6.B, R15.2; no longer LED5.A, R4.1
- net N$7: now also Q8.B, R16.2; no longer LED5.C, Q2.C
- net N$8: now also Q7.B, R17.2; no longer Q1.B, R5.1
- net N$9: now also Q3.B, R21.2; no longer Q2.B, R11.1
- net UART_RX: now also MAIN_CHIP.34, R1.1; no longer IC1.34, R6.1
- net UART_TX: now also MAIN_CHIP.35, R4.1; no longer IC1.35, R10.1
- net VBAT: now also C2.+, X3-1.KL; no longer C3.+, X4-2.KL
- net XBEERX: now also JP1.3, R3.1, R4.2; no longer R10.2, R9.1, X2-3.1
- net XBEETX: now also JP1.2, R1.2; no longer R6.2, X2-2.1
Other:
- note added: "2. Processors"
- note added: "3. XBEE"
- note added: "4. Connectors"
- note added: "5. Power Supply"
- note added: "6. LEDs"
- note added: "Connectors"
- note added: "LEDs"
- note added: "Power Supply"
- note added: "Processors"
- note added: "XBEE"
- note removed: "2 uC - Power"
- note removed: "3 XBEE - Display - Connectors"
- note removed: "Remote Control"
- note removed: "XBEE - Display"
- note removed: "uC - Power - Connectors"
